File: hardware/iv-grapher.sch (KiCad schematic (older format))
At the start: 74 parts, among them IC1 TC7660SO-08, P1 DUT, P2 CONN_02X06, P3 POWER, Q1 IRLML6244, Q2 IRLML6244, U1 MCP4921-E/SN, U2 LM358, U3 MCP3302, U4 MC78L18ACP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

Commit message: Start of design version 2
Parts:
- removed R1, R3, R5, R7: 100k, Resistors_SMD:R_0805, symbol R
- added U?: AD620, symbol AD620
- D2, D3: value 5V1 -> 5V6
Connections:
- net DUT+: now also U?.3 (+)
- net DUT-: now also U?.2 (-)
- net GND: now also U?.5 (Ref); no longer U3.2 (CH1), U3.4 (CH3)
- net VCC: now also U?.7 (V+); no longer U2.8 (V+)
- net VEE: now also U?.4 (V-); no longer U2.4 (V-)
- net at U2.7: no longer R4.2
- net at U5.5 (CII): now also R13.2, R14.1; no longer R13.1
- net at C10.1, C11.1, C9.1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: now also R13.1; no longer R13.2, R14.1
- new net: R4.2, U?.6
- no-connect marks 2 -> 4
Other:
- note removed: "This divider is completely wrong. Redesign and redo PCB"
- moved on the sheet: R13, U2B
Changed lines of the file:
@@
 L LM358 U2
 U 2 1 58B6B6D3
-P 6000 1400
-F 0 "U2" H 6000 1600 50  0000 L CNN
-F 1 "LM358" H 6000 1200 50  0000 L CNN
-F 2 "Housings_SOIC:SOIC-8_3.9x4.9mm_Pitch1.27mm" H 6000 1400 50  0001 C CNN
-F 3 "" H 6000 1400 50  0000 C CNN
-	2    6000 1400
-	1    0    0    -1
-$EndComp
-$Comp
-L R R3
-U 1 1 58B6B732
-P 5250 1300
-F 0 "R3" V 5330 1300 50  0000 C CNN
-F 1 "100k" V 5250 1300 50  0000 C CNN
-F 2 "Resistors_SMD:R_0805" V 5180 1300 50  0001 C CNN
-F 3 "" H 5250 1300 50  0000 C CNN
-	1    5250 1300
-	0    1    1    0
-$EndComp
-$Comp
-L R R5
-U 1 1 58B6B7AB
-P 5250 1500
-F 0 "R5" V 5330 1500 50  0000 C CNN
-F 1 "100k" V 5250 1500 50  0000 C CNN
-F 2 "Resistors_SMD:R_0805" V 5180 1500 50  0001 C CNN
-F 3 "" H 5250 1500 50  0000 C CNN
-	1    5250 1500
-	0    1    1    0
-$EndComp
-$Comp
-L R R7
-U 1 1 58B6BBB0
-P 5550 1800
-F 0 "R7" V 5630 1800 50  0000 C CNN
-F 1 "100k" V 5550 1800 50  0000 C CNN
-F 2 "Resistors_SMD:R_0805" V 5480 1800 50  0001 C CNN
-F 3 "" H 5550 1800 50  0000 C CNN
-	1    5550 1800
-	1    0    0    -1
-$EndComp
-$Comp
-L R R1
-U 1 1 58B6BC05
-P 5550 1000
-F 0 "R1" V 5630 1000 50  0000 C CNN
-F 1 "100k" V 5550 1000 50  0000 C CNN
-F 2 "Resistors_SMD:R_0805" V 5480 1000 50  0001 C CNN
-F 3 "" H 5550 1000 50  0000 C CNN
-	1    5550 1000
+P 6750 3350
+F 0 "U2" H 6750 3550 50  0000 L CNN
+F 1 "LM358" H 6750 3150 50  0000 L CNN
+F 2 "Housings_SOIC:SOIC-8_3.9x4.9mm_Pitch1.27mm" H 6750 3350 50  0001 C CNN
+F 3 "" H 6750 3350 50  0000 C CNN
+	2    6750 3350
 	1    0    0    -1
 $EndComp
@@
 $EndComp
 $Comp
-L GND #PWR03
-U 1 1 58B6D30E
-P 5550 750
-F 0 "#PWR03" H 5550 500 50  0001 C CNN
-F 1 "GND" H 5550 600 50  0000 C CNN
-F 2 "" H 5550 750 50  0000 C CNN
-F 3 "" H 5550 750 50  0000 C CNN
-	1    5550 750
-	-1   0    0    1
-$EndComp
-$Comp
 L TC7660SO-08 IC1
 U 1 1 58B6F7C2
@@
 P 7500 1750
 F 0 "D2" H 7500 1850 50  0000 C CNN
-F 1 "5V1" H 7500 1650 50  0000 C CNN
+F 1 "5V6" H 7500 1650 50  0000 C CNN
 F 2 "Diodes_SMD:SOD-123" H 7500 1750 50  0001 C CNN
 F 3 "" H 7500 1750 50  0000 C CNN
@@
 L VEE #PWR012
 U 1 1 58B87071
-P 5900 1750
-F 0 "#PWR012" H 5900 1600 50  0001 C CNN
-F 1 "VEE" H 5900 1900 50  0000 C CNN
-F 2 "" H 5900 1750 50  0000 C CNN
-F 3 "" H 5900 1750 50  0000 C CNN
-	1    5900 1750
+P 5250 1750
+F 0 "#PWR012" H 5250 1600 50  0001 C CNN
+F 1 "VEE" H 5250 1900 50  0000 C CNN
+F 2 "" H 5250 1750 50  0000 C CNN
+F 3 "" H 5250 1750 50  0000 C CNN
+	1    5250 1750
 	-1   0    0    1
 $EndComp
@@
 L VCC #PWR013
 U 1 1 58B87340
-P 5900 1050
-F 0 "#PWR013" H 5900 900 50  0001 C CNN
-F 1 "VCC" H 5900 1200 50  0000 C CNN
-F 2 "" H 5900 1050 50  0000 C CNN
-F 3 "" H 5900 1050 50  0000 C CNN
-	1    5900 1050
+P 5250 1050
+F 0 "#PWR013" H 5250 900 50  0001 C CNN
+F 1 "VCC" H 5250 1200 50  0000 C CNN
+F 2 "" H 5250 1050 50  0000 C CNN
+F 3 "" H 5250 1050 50  0000 C CNN
+	1    5250 1050
 	1    0    0    -1
 $EndComp
@@
 $EndComp
 $Comp
-L GND #PWR017
-U 1 1 58B9DE6D
-P 8050 1550
-F 0 "#PWR017" H 8050 1300 50  0001 C CNN
-F 1 "GND" H 8050 1400 50  0000 C CNN
-F 2 "" H 8050 1550 50  0000 C CNN
-F 3 "" H 8050 1550 50  0000 C CNN
-	1    8050 1550
-	0    1    1    0
-$EndComp
-$Comp
-L GND #PWR018
-U 1 1 58B9DEB5
-P 8050 1850
-F 0 "#PWR018" H 8050 1600 50  0001 C CNN
-F 1 "GND" H 8050 1700 50  0000 C CNN
-F 2 "" H 8050 1850 50  0000 C CNN
-F 3 "" H 8050 1850 50  0000 C CNN
-	1    8050 1850
-	0    1    1    0
-$EndComp
-$Comp
 L GND #PWR019
 U 1 1 58B9E9DB
@@
 L R R13
 U 1 1 58BA2250
-P 1400 4950
-F 0 "R13" V 1480 4950 50  0000 C CNN
-F 1 "18k" V 1400 4950 50  0000 C CNN
-F 2 "Resistors_SMD:R_0805" V 1330 4950 50  0001 C CNN
-F 3 "" H 1400 4950 50  0000 C CNN
-	1    1400 4950
-	1    0    0    -1
+P 1650 5200
+F 0 "R13" V 1730 5200 50  0000 C CNN
+F 1 "18k" V 1650 5200 50  0000 C CNN
+F 2 "Resistors_SMD:R_0805" V 1580 5200 50  0001 C CNN
+F 3 "" H 1650 5200 50  0000 C CNN
+	1    1650 5200
+	0    1    1    0
 $EndComp
 $Comp
@@
 	1    0    0    -1
 $EndComp
-Text Notes 1500 5200 0    60   ~ 0
+Text Notes 1500 5100 0    60   ~ 0
 33k + 2k = 21.9v\n15k + 1k = 20v
 $Comp
@@
 	4950 1700 4950 1500
 Wire Wire Line
-	4950 1500 5100 1500
-Wire Wire Line
-	5100 1300 4950 1300
+	4950 1500 5050 1500
+Wire Wire Line
+	4950 1300 5050 1300
 Wire Wire Line
 	4950 1300 4950 1200
@@
 	4950 1200 4300 1200
 Wire Wire Line
-	5400 1300 5700 1300
-Wire Wire Line
-	5400 1500 5700 1500
-Wire Wire Line
-	5550 1150 5550 1300
-Connection ~ 5550 1300
-Wire Wire Line
-	5550 1650 5550 1500
-Connection ~ 5550 1500
-Wire Wire Line
-	6300 1400 6600 1400
-Connection ~ 6450 1400
+	5650 1400 6600 1400
 Wire Wire Line
 	7100 2450 7100 2550
@@
 Connection ~ 4450 6600
 Wire Wire Line
-	5900 1750 5900 1700
+	5250 1750 5250 1700
 Wire Wire Line
 	3550 1750 3550 1700
 Wire Wire Line
-	5900 1100 5900 1050
+	5250 1100 5250 1050
 Wire Wire Line
 	3550 1100 3550 1050
@@
 Connection ~ 4300 2100
 Wire Wire Line
-	8050 1850 8150 1850
-Wire Wire Line
-	8150 1550 8050 1550
-Wire Wire Line
 	9900 900  9900 1000
 Wire Wire Line
@@
 	4400 3700 4400 5200
 Wire Wire Line
-	4400 5200 1400 5200
+	4400 5200 1800 5200
 Connection ~ 4250 4050
 Wire Wire Line
 	1400 5700 1400 5600
 Wire Wire Line
-	1400 5100 1400 5300
+	1400 4700 1400 5300
 Connection ~ 1400 5200
 Wire Wire Line
 	850  5100 850  5000
-Wire Wire Line
-	1400 4800 1400 4700
 Connection ~ 4400 4050
 Wire Wire Line
@@
 	5400 3700 4950 3700
 Wire Wire Line
-	4750 3700 4400 3700
+	4400 3700 4750 3700
 Wire Wire Line
 	1050 6450 950  6450
@@
 P 7800 3100
 F 0 "D3" H 7800 3200 50  0000 C CNN
-F 1 "5V1" H 7800 3000 50  0000 C CNN
+F 1 "5V6" H 7800 3000 50  0000 C CNN
 F 2 "Diodes_SMD:SOD-123" H 7800 3100 50  0001 C CNN
 F 3 "" H 7800 3100 50  0000 C CNN
@@
 	5100 2850 5100 2100
 Wire Wire Line
-	5550 850  5550 750
-Wire Wire Line
-	5550 1950 5550 2050
-Wire Wire Line
-	5550 2050 6450 2050
-Wire Wire Line
-	6450 2050 6450 1400
-Text Notes 1450 5350 0    60   ~ 0
-This divider is completely wrong. Redesign and redo PCB
+	1500 5200 1400 5200
+$Comp
+L AD620 U?
+U 1 1 58DE9AD2
+P 5350 1400
+F 0 "U?" H 5550 1550 50  0000 L CNN
+F 1 "AD620" H 5550 1250 50  0000 L CNN
+F 2 "" H 5350 1400 50  0000 C CNN
+F 3 "" H 5350 1400 50  0000 C CNN
+	1    5350 1400
+	1    0    0    -1
+$EndComp
+$Comp
+L GND #PWR?
+U 1 1 58DEB3A5
+P 5350 1050
+F 0 "#PWR?" H 5350 800 50  0001 C CNN
+F 1 "GND" H 5350 900 50  0000 C CNN
+F 2 "" H 5350 1050 50  0000 C CNN
+F 3 "" H 5350 1050 50  0000 C CNN
+	1    5350 1050
+	-1   0    0    1
+$EndComp
+Wire Wire Line
+	5350 1050 5350 1100
+NoConn ~ 5350 1700
+NoConn ~ 5450 1700
 $EndSCHEMATC
